Commit message: fixes to the robot to make it work right.

File: urdf/macros.xacro (robot description, xacro)
@@ -25,7 +25,17 @@
       <parent link="base_link"/>
       <child link="${prefix}_wheel"/>
-      <origin xyz="${x} ${y} 0" rpy="${pi/2} 0 0"/>
+      <origin xyz="${x} ${y} ${-base_height/2}" rpy="${pi/2} 0 0"/>  <!-- Corrected RPY and Z offset -->
       <axis xyz="0 0 1"/>
     </joint>
+    <transmission name="${prefix}_wheel_transmission">
+      <type>transmission_interface/SimpleTransmission</type>
+      <joint name="${prefix}_wheel_joint">
+        <hardwareInterface>hardware_interface/VelocityJointInterface</hardwareInterface>
+      </joint>
+      <actuator name="${prefix}_wheel_motor">
+        <hardwareInterface>hardware_interface/VelocityJointInterface</hardwareInterface>
+        <mechanicalReduction>1</mechanicalReduction>
+      </actuator>
+    </transmission>
   </xacro:macro>
   <!-- Caster Wheel Macro -->
@@ -53,5 +63,5 @@
       <parent link="base_link"/>
       <child link="caster_wheel"/>
-      <origin xyz="${base_length/2 - caster_radius} 0 -${caster_radius}"/>
+      <origin xyz="${base_length/2 - caster_radius} 0 ${-base_height/2 - caster_radius}"/>  <!-- Corrected Z offset for caster wheel -->
     </joint>
   </xacro:macro>
@@ -80,7 +90,7 @@
       <parent link="base_link"/>
       <child link="${prefix}_arm"/>
-      <origin xyz="${base_length/2} ${side_mult * 0.1} ${base_height/2}"/>
+      <origin xyz="${base_length/2} ${side_mult * base_width/2} ${base_height/2 + arm_radius}"/>  <!-- Corrected Z offset for arm joint -->
       <axis xyz="0 1 0"/>
-      <limit lower="-0.05" upper="0.05" effort="100" velocity="1"/>
+      <limit lower="${-arm_length/2}" upper="${arm_length/2}" effort="100" velocity="1"/>  <!-- Adjusted limits for arm movement -->
     </joint>
     <!-- Gripper -->

File: urdf/properties.xacro (robot description, xacro)
@@ -2,11 +2,13 @@
 <robot xmlns:xacro="http://www.ros.org/wiki/xacro">
   <!-- Robot Properties -->
-  <xacro:property name="base_width" value="0.4"/>
-  <xacro:property name="base_length" value="0.6"/>
-  <xacro:property name="base_height" value="0.1"/>
-  <xacro:property name="wheel_radius" value="0.1"/>
-  <xacro:property name="wheel_width" value="0.05"/>
-  <xacro:property name="caster_radius" value="0.05"/>
-  <xacro:property name="arm_length" value="0.4"/>
-  <xacro:property name="arm_radius" value="0.03"/>
+  <xacro:property name="scaling_factor" value="0.5" />
+  <xacro:property name="arm_offset_z" value="0.02 * scaling_factor"/>
+  <xacro:property name="base_width" value="${0.4 * scaling_factor}"/>
+  <xacro:property name="base_length" value="${0.6 * scaling_factor}"/>
+  <xacro:property name="base_height" value="${0.1 * scaling_factor}"/>
+  <xacro:property name="wheel_radius" value="${0.1 * scaling_factor}"/>
+  <xacro:property name="wheel_width" value="${0.05 * scaling_factor}"/>
+  <xacro:property name="caster_radius" value="${0.05 * scaling_factor}"/>
+  <xacro:property name="arm_length" value="${0.2 * scaling_factor}"/>
+  <xacro:property name="arm_radius" value="${0.03 * scaling_factor}"/>
 </robot>

File: urdf/three_wheeled_robot.xacro (robot description, xacro)
@@ -29,6 +29,8 @@
   </link>
   <!-- Add wheels -->
-  <xacro:wheel prefix="left" x="-0.2" y="${base_width/2 + wheel_width/2}"/>
-  <xacro:wheel prefix="right" x="-0.2" y="-${base_width/2 + wheel_width/2}"/>
+  <!-- <xacro:wheel prefix="left" x="0" y="${base_width/2}"/>
+  <xacro:wheel prefix="right" x="0" y="-${base_width/2}"/> -->
+  <xacro:wheel prefix="left" x="${-base_length/2 + wheel_radius}" y="${base_width/2 + wheel_radius/4}"/>
+  <xacro:wheel prefix="right" x="${-base_length/2 + wheel_radius}" y="${-base_width/2 - wheel_radius/4}"/>
   <!-- Add caster wheel -->
   <xacro:caster_wheel />
