Commit message: make wheels fatter

File: urdf/properties.xacro (robot description, xacro)
@@ -8,6 +8,6 @@
   <xacro:property name="base_height" value="${0.1 * scaling_factor}"/>
   <xacro:property name="wheel_radius" value="${0.1 * scaling_factor}"/>
-  <xacro:property name="wheel_width" value="${0.05 * scaling_factor}"/>
-  <xacro:property name="caster_radius" value="${0.05 * scaling_factor}"/>
+  <xacro:property name="wheel_width" value="${0.1 * scaling_factor}"/>
+  <xacro:property name="caster_radius" value="${0.1 * scaling_factor}"/>
   <xacro:property name="arm_length" value="${0.2 * scaling_factor}"/>
   <xacro:property name="arm_radius" value="${0.03 * scaling_factor}"/>

Commit message: remove scaling factor. unnecessary complexity

File: urdf/properties.xacro (robot description, xacro)
@@ -2,13 +2,11 @@
 <robot xmlns:xacro="http://www.ros.org/wiki/xacro">
   <!-- Robot Properties -->
-  <xacro:property name="scaling_factor" value="0.5" />
-  <xacro:property name="arm_offset_z" value="0.02 * scaling_factor"/>
-  <xacro:property name="base_width" value="${0.4 * scaling_factor}"/>
-  <xacro:property name="base_length" value="${0.6 * scaling_factor}"/>
-  <xacro:property name="base_height" value="${0.2 * scaling_factor}"/>
-  <xacro:property name="wheel_radius" value="${0.1 * scaling_factor}"/>
-  <xacro:property name="wheel_width" value="${0.08 * scaling_factor}"/>
-  <xacro:property name="caster_radius" value="${0.05 * scaling_factor}"/>
-  <xacro:property name="arm_length" value="${0.2 * scaling_factor}"/>
-  <xacro:property name="arm_radius" value="${0.03 * scaling_factor}"/>
+  <xacro:property name="base_width" value="0.2"/>
+  <xacro:property name="base_length" value="0.3"/>
+  <xacro:property name="base_height" value="0.1"/>
+  <xacro:property name="wheel_radius" value="0.05"/>
+  <xacro:property name="wheel_width" value="0.04"/>
+  <xacro:property name="caster_radius" value="0.025"/>
+  <xacro:property name="arm_length" value="0.1"/>
+  <xacro:property name="arm_radius" value="0.015"/>
 </robot>

Commit message: reduce width of robot for more convenient movement

File: urdf/properties.xacro (robot description, xacro)
@@ -2,5 +2,5 @@
 <robot xmlns:xacro="http://www.ros.org/wiki/xacro">
   <!-- Robot Properties -->
-  <xacro:property name="base_width" value="0.4"/>
+  <xacro:property name="base_width" value="0.31"/>
   <xacro:property name="base_length" value="0.35"/>
   <xacro:property name="base_height" value="0.1"/>
