Commit message: committing changes before they're lost forever

File: urdf/gazebo.xacro (robot description, xacro)
@@ -3,22 +3,12 @@
   <!-- ROS Control plugin -->
   <gazebo>
-    <plugin name="gazebo_ros_control" filename="libgazebo_ros_control.so">
-      <robotNamespace>/three_wheeled_robot</robotNamespace>
-    </plugin>
-  </gazebo>
-  <!-- Differential drive plugin -->
-  <gazebo>
-    <plugin name="differential_drive_controller" filename="libgazebo_ros_diff_drive.so">
+    <plugin name="diff_drive_controller" filename="libgazebo_ros_diff_drive.so">
+      <robotNamespace>/</robotNamespace>
+      <commandTopic>cmd_vel</commandTopic>
+      <odometryTopic>odom</odometryTopic>
+      <odometryFrame>odom</odometryFrame>
+      <robotBaseFrame>base_link</robotBaseFrame>
       <leftJoint>left_wheel_joint</leftJoint>
       <rightJoint>right_wheel_joint</rightJoint>
-      <wheelSeparation>${base_width + wheel_width}</wheelSeparation>
-      <wheelDiameter>${2 * wheel_radius}</wheelDiameter>
-      <robotBaseFrame>base_link</robotBaseFrame>
-      <publishWheelTF>true</publishWheelTF>
-      <publishWheelJointState>true</publishWheelJointState>
-      <wheelAcceleration>1</wheelAcceleration>
-      <wheelTorque>20</wheelTorque>
-      <odometrySource>world</odometrySource>
-      <publishOdomTF>true</publishOdomTF>
     </plugin>
   </gazebo>

File: urdf/macros.xacro (robot description, xacro)
@@ -18,5 +18,5 @@
       </collision>
       <inertial>
-        <mass value="1.0"/>
+        <mass value="0.5"/>
         <inertia ixx="0.0001" ixy="0" ixz="0" iyy="0.0001" iyz="0" izz="0.0001"/>
       </inertial>
@@ -28,14 +28,4 @@
       <axis xyz="0 0 1"/>
     </joint>
-    <transmission name="${prefix}_wheel_transmission">
-      <type>transmission_interface/SimpleTransmission</type>
-      <joint name="${prefix}_wheel_joint">
-        <hardwareInterface>hardware_interface/VelocityJointInterface</hardwareInterface>
-      </joint>
-      <actuator name="${prefix}_wheel_motor">
-        <hardwareInterface>hardware_interface/VelocityJointInterface</hardwareInterface>
-        <mechanicalReduction>1</mechanicalReduction>
-      </actuator>
-    </transmission>
   </xacro:macro>
   <!-- Caster Wheel Macro -->
@@ -83,14 +73,14 @@
       </collision>
       <inertial>
-        <mass value="1.0"/>
+        <mass value="0.25"/>
         <inertia ixx="0.0001" ixy="0" ixz="0" iyy="0.0001" iyz="0" izz="0.0001"/>
       </inertial>
     </link>
-    <joint name="${prefix}_arm_joint" type="prismatic">
+    <joint name="${prefix}_arm_joint" type="fixed">
       <parent link="base_link"/>
       <child link="${prefix}_arm"/>
       <origin xyz="${base_length/2} ${side_mult * base_width/2} ${base_height/2 + arm_radius}"/>  <!-- Corrected Z offset for arm joint -->
       <axis xyz="0 1 0"/>
-      <limit lower="${-arm_length/2}" upper="${arm_length/2}" effort="100" velocity="1"/>  <!-- Adjusted limits for arm movement -->
+      <!-- <limit lower="${-arm_length/2}" upper="${arm_length/2}" effort="100" velocity="1"/>  --><!-- Adjusted limits for arm movement -->
     </joint>
     <!-- Gripper -->
@@ -110,5 +100,5 @@
       </collision>
       <inertial>
-        <mass value="0.3"/>
+        <mass value="0.2"/>
         <inertia ixx="0.00005" ixy="0" ixz="0" iyy="0.0005" iyz="0" izz="0.00005"/>
       </inertial>

File: urdf/three_wheeled_robot.xacro (robot description, xacro)
@@ -24,5 +24,5 @@
     </collision>
     <inertial>
-      <mass value="5.0"/>
+      <mass value="1.5"/>
       <inertia ixx="0.0833" ixy="0" ixz="0" iyy="0.0833" iyz="0" izz="0.1667"/>
     </inertial>

Commit message: major changes: dimensions, gazebo settings and locations of wheels

File: urdf/gazebo.xacro (robot description, xacro)
@@ -11,5 +11,17 @@
       <leftJoint>left_wheel_joint</leftJoint>
       <rightJoint>right_wheel_joint</rightJoint>
+      <wheelSeparation>${base_width}</wheelSeparation>
+      <legacyMode>false</legacyMode>
+      <wheelDiameter>${2 * wheel_radius}</wheelDiameter>
+      <robotBaseFrame>base_link</robotBaseFrame>
+      <publishOdomTF>true</publishOdomTF>
+      <publishWheelJointState>true</publishWheelJointState>
+      <wheelAcceleration>1</wheelAcceleration>
+      <wheelTorque>20</wheelTorque>
+      <updateRate>50</updateRate>
     </plugin>
   </gazebo>
+  <material name="orange">
+    <color rgba="1.0 0.423529411765 0.0392156862745 1.0"/>
+  </material>
 </robot>

File: urdf/macros.xacro (robot description, xacro)
@@ -19,5 +19,5 @@
       <inertial>
         <mass value="0.5"/>
-        <inertia ixx="0.0001" ixy="0" ixz="0" iyy="0.0001" iyz="0" izz="0.0001"/>
+        <inertia ixx="0.001" ixy="0" ixz="0" iyy="0.001" iyz="0" izz="0.001"/>
       </inertial>
     </link>
@@ -25,5 +25,5 @@
       <parent link="base_link"/>
       <child link="${prefix}_wheel"/>
-      <origin xyz="${x} ${y} ${-base_height/2}" rpy="${pi/2} 0 0"/>  <!-- Corrected RPY and Z offset -->
+      <origin xyz="${x} ${y * (base_width/2 + wheel_radius/2)} ${-base_height/3}" rpy="${pi/2} 0 0"/>  <!-- Corrected RPY and Z offset -->
       <axis xyz="0 0 1"/>
     </joint>
@@ -34,5 +34,5 @@
       <visual>
         <geometry>
-          <sphere radius="${caster_radius}"/>
+          <sphere radius="${wheel_radius}"/>
         </geometry>
         <material name="grey">
@@ -53,5 +53,5 @@
       <parent link="base_link"/>
       <child link="caster_wheel"/>
-      <origin xyz="${base_length/2 - caster_radius} 0 ${-base_height/2 - caster_radius}"/>  <!-- Corrected Z offset for caster wheel -->
+      <origin xyz="${base_length/3.3} 0 ${-(base_height/3)}" rpy="0 0 0"/>  <!-- Corrected Z offset for caster wheel -->
     </joint>
   </xacro:macro>

File: urdf/properties.xacro (robot description, xacro)
@@ -6,8 +6,8 @@
   <xacro:property name="base_width" value="${0.4 * scaling_factor}"/>
   <xacro:property name="base_length" value="${0.6 * scaling_factor}"/>
-  <xacro:property name="base_height" value="${0.1 * scaling_factor}"/>
+  <xacro:property name="base_height" value="${0.2 * scaling_factor}"/>
   <xacro:property name="wheel_radius" value="${0.1 * scaling_factor}"/>
-  <xacro:property name="wheel_width" value="${0.1 * scaling_factor}"/>
-  <xacro:property name="caster_radius" value="${0.1 * scaling_factor}"/>
+  <xacro:property name="wheel_width" value="${0.08 * scaling_factor}"/>
+  <xacro:property name="caster_radius" value="${0.05 * scaling_factor}"/>
   <xacro:property name="arm_length" value="${0.2 * scaling_factor}"/>
   <xacro:property name="arm_radius" value="${0.03 * scaling_factor}"/>

File: urdf/three_wheeled_robot.xacro (robot description, xacro)
@@ -10,4 +10,6 @@
   <!-- Base Link -->
   <link name="base_link">
+    <pose>0.2 0.1 ${base_height/2} 0 0 0.15</pose>
+    <origin xyz="0.2 0.1 ${base_height/2}" rpy="0 0 0"/>
     <visual>
       <geometry>
@@ -24,17 +26,10 @@
     </collision>
     <inertial>
-      <mass value="1.5"/>
-      <inertia ixx="0.0833" ixy="0" ixz="0" iyy="0.0833" iyz="0" izz="0.1667"/>
+      <mass value="5"/>
+      <inertia ixx="0.1" ixy="0" ixz="0" iyy="0.1" iyz="0" izz="0.1667"/>
     </inertial>
   </link>
-  <!-- Add wheels -->
-  <!-- <xacro:wheel prefix="left" x="0" y="${base_width/2}"/>
-  <xacro:wheel prefix="right" x="0" y="-${base_width/2}"/> -->
-  <xacro:wheel prefix="left" x="${-base_length/2 + wheel_radius}" y="${base_width/2 + wheel_radius/4}"/>
-  <xacro:wheel prefix="right" x="${-base_length/2 + wheel_radius}" y="${-base_width/2 - wheel_radius/4}"/>
-  <!-- Add caster wheel -->
   <xacro:caster_wheel />
-  <!-- Add arms -->
-  <xacro:arm prefix="left" side_mult="1"/>
-  <xacro:arm prefix="right" side_mult="-1"/>
+  <xacro:wheel prefix="left" x="${-base_length/2 + wheel_radius}" y="1"/>
+  <xacro:wheel prefix="right" x="${-base_length/2 + wheel_radius}" y="-1"/>
 </robot>

Commit message: From googling and testing - this reduces bouncing - a bit.

File: urdf/gazebo.xacro (robot description, xacro)
@@ -17,5 +17,7 @@
       <publishOdomTF>true</publishOdomTF>
       <publishWheelJointState>true</publishWheelJointState>
+      <max_wheel_torque>20</max_wheel_torque>
       <wheelAcceleration>1</wheelAcceleration>
+      <max_wheel_acceleration>1</max_wheel_acceleration>
       <wheelTorque>20</wheelTorque>
       <updateRate>50</updateRate>
@@ -25,3 +27,29 @@
     <color rgba="1.0 0.423529411765 0.0392156862745 1.0"/>
   </material>
+  <material name="black">
+    <color rgba="0 0 0 1"/>
+  </material>
+  <gazebo reference="caster_wheel">
+    <mu1 value="1.0"/>
+    <mu2 value="1.0"/>
+    <kp  value="10000000.0" />
+    <kd  value="1.0" />
+    <material>Gazebo/Orange</material>
+  </gazebo>
+  <gazebo reference="right_wheel">
+    <mu1 value="1.0"/>
+    <mu2 value="1.0"/>
+    <kp  value="10000000.0" />
+    <kd  value="1.0" />
+    <fdir1 value="1 0 0"/>
+    <material>Gazebo/Black</material>
+  </gazebo>
+  <gazebo reference="left_wheel">
+    <mu1 value="1.0"/>
+    <mu2 value="1.0"/>
+    <kp  value="10000000.0" />
+    <kd  value="1.0" />
+    <fdir1 value="1 0 0"/>
+    <material>Gazebo/Black</material>
+  </gazebo>
 </robot>

Commit message: 2 days later the robots moves are stable!

File: urdf/gazebo.xacro (robot description, xacro)
@@ -22,4 +22,5 @@
       <wheelTorque>20</wheelTorque>
       <updateRate>50</updateRate>
+      <max_velocity>0.5</max_velocity>
     </plugin>
   </gazebo>
@@ -38,6 +39,6 @@
   </gazebo>
   <gazebo reference="right_wheel">
-    <mu1 value="1.0"/>
-    <mu2 value="1.0"/>
+    <mu1 value="1.5"/>
+    <mu2 value="1.5"/>
     <kp  value="10000000.0" />
     <kd  value="1.0" />
@@ -46,6 +47,6 @@
   </gazebo>
   <gazebo reference="left_wheel">
-    <mu1 value="1.0"/>
-    <mu2 value="1.0"/>
+    <mu1 value="1.5"/>
+    <mu2 value="1.5"/>
     <kp  value="10000000.0" />
     <kd  value="1.0" />

File: urdf/macros.xacro (robot description, xacro)
@@ -14,10 +14,10 @@
       <collision>
         <geometry>
-          <cylinder radius="${wheel_radius}" length="${wheel_width}"/>
+          <cylinder radius="${wheel_radius}" length="${2 * wheel_width}"/>
         </geometry>
       </collision>
       <inertial>
-        <mass value="0.5"/>
-        <inertia ixx="0.001" ixy="0" ixz="0" iyy="0.001" iyz="0" izz="0.001"/>
+        <mass value="1"/>
+        <inertia ixx="0.0007" ixy="0" ixz="0" iyy="0.0007" iyz="0" izz="0.0007"/>
       </inertial>
     </link>
@@ -25,6 +25,7 @@
       <parent link="base_link"/>
       <child link="${prefix}_wheel"/>
-      <origin xyz="${x} ${y * (base_width/2 + wheel_radius/2)} ${-base_height/3}" rpy="${pi/2} 0 0"/>  <!-- Corrected RPY and Z offset -->
-      <axis xyz="0 0 1"/>
+      <origin xyz="${x} ${y * (base_width/2 + wheel_radius/2)} 0" rpy="${pi/2} 0 0"/>  <!-- Corrected RPY and Z offset -->
+      <axis xyz="0 0 -1"/>
+      <joint_properties damping="0.5" friction="0.5"/>
     </joint>
   </xacro:macro>
@@ -34,5 +35,5 @@
       <visual>
         <geometry>
-          <sphere radius="${wheel_radius}"/>
+          <sphere radius="${caster_radius}"/>
         </geometry>
         <material name="grey">
@@ -46,6 +47,7 @@
       </collision>
       <inertial>
-        <mass value="0.5"/>
-        <inertia ixx="0.0001" ixy="0" ixz="0" iyy="0.0001" iyz="0" izz="0.0001"/>
+        <mass value="0.3"/>
+        <inertia ixx="0.00018" ixy="0" ixz="0" iyy="0.00018" iyz="0" izz="0.00018"/>
+        <origin xyz="0 0 0" rpy="0 0 0" />
       </inertial>
     </link>
@@ -53,5 +55,6 @@
       <parent link="base_link"/>
       <child link="caster_wheel"/>
-      <origin xyz="${base_length/3.3} 0 ${-(base_height/3)}" rpy="0 0 0"/>  <!-- Corrected Z offset for caster wheel -->
+      <origin xyz="${base_length/3.3} 0 ${-caster_radius}" rpy="0 0 0"/>  <!-- Corrected Z offset for caster wheel -->
+      <dynamics damping="0.01"/>
     </joint>
   </xacro:macro>
@@ -80,5 +83,5 @@
       <parent link="base_link"/>
       <child link="${prefix}_arm"/>
-      <origin xyz="${base_length/2} ${side_mult * base_width/2} ${base_height/2 + arm_radius}"/>  <!-- Corrected Z offset for arm joint -->
+      <origin xyz="${base_length/2} ${side_mult * (base_width /2 - 0.005)} 0.04"/>  <!-- Corrected Z offset for arm joint -->
       <axis xyz="0 1 0"/>
       <!-- <limit lower="${-arm_length/2}" upper="${arm_length/2}" effort="100" velocity="1"/>  --><!-- Adjusted limits for arm movement -->
@@ -88,5 +91,5 @@
       <visual>
         <geometry>
-          <box size="${arm_length} 0.05 0.05"/>
+          <box size="${arm_length} 0.02 0.08"/>
         </geometry>
         <material name="grey">
@@ -96,5 +99,5 @@
       <collision>
         <geometry>
-          <box size="${arm_length} 0.05 0.05"/>
+          <box size="${arm_length} 0.02 0.08"/>
         </geometry>
       </collision>

File: urdf/properties.xacro (robot description, xacro)
@@ -2,10 +2,10 @@
 <robot xmlns:xacro="http://www.ros.org/wiki/xacro">
   <!-- Robot Properties -->
-  <xacro:property name="base_width" value="0.2"/>
-  <xacro:property name="base_length" value="0.3"/>
+  <xacro:property name="base_width" value="0.4"/>
+  <xacro:property name="base_length" value="0.35"/>
   <xacro:property name="base_height" value="0.1"/>
-  <xacro:property name="wheel_radius" value="0.05"/>
+  <xacro:property name="wheel_radius" value="0.07"/>
   <xacro:property name="wheel_width" value="0.04"/>
-  <xacro:property name="caster_radius" value="0.025"/>
+  <xacro:property name="caster_radius" value="0.02"/>
   <xacro:property name="arm_length" value="0.1"/>
   <xacro:property name="arm_radius" value="0.015"/>

File: urdf/three_wheeled_robot.xacro (robot description, xacro)
@@ -10,9 +10,8 @@
   <!-- Base Link -->
   <link name="base_link">
-    <pose>0.2 0.1 ${base_height/2} 0 0 0.15</pose>
     <origin xyz="0.2 0.1 ${base_height/2}" rpy="0 0 0"/>
     <visual>
       <geometry>
-        <box size="${base_length} ${base_width} ${base_height}"/>
+        <box size="${base_length} ${base_width} ${base_height/2}"/>
       </geometry>
       <material name="blue">
@@ -26,10 +25,13 @@
     </collision>
     <inertial>
-      <mass value="5"/>
-      <inertia ixx="0.1" ixy="0" ixz="0" iyy="0.1" iyz="0" izz="0.1667"/>
+      <mass value="0.6"/>
+      <inertia ixx="0.001" ixy="0" ixz="0" iyy="0.001" iyz="0" izz="0.001"/>
+      <origin xyz="0 0 0" rpy="0 0 0"/>
     </inertial>
   </link>
   <xacro:caster_wheel />
-  <xacro:wheel prefix="left" x="${-base_length/2 + wheel_radius}" y="1"/>
-  <xacro:wheel prefix="right" x="${-base_length/2 + wheel_radius}" y="-1"/>
+  <xacro:wheel prefix="left" x="${-base_length/3}" y="1"/>
+  <xacro:wheel prefix="right" x="${-base_length/3}" y="-1"/>
+  <xacro:arm prefix="left" side_mult="1"/>
+  <xacro:arm prefix="right" side_mult="-1"/>
 </robot>

Commit message: T-30h and the robot is working!!!!

File: urdf/gazebo.xacro (robot description, xacro)
@@ -31,4 +31,13 @@
     <color rgba="0 0 0 1"/>
   </material>
+  <gazebo reference="base_link">
+    <material>Gazebo/Blue</material>
+    <mu1 value="1.0"/>
+    <mu2 value="1.0"/>
+    <kp  value="10000000.0"/>
+    <kd  value="100.0"/>
+    <maxVel>0.0</maxVel>
+    <minDepth>0.001</minDepth>
+  </gazebo>
   <gazebo reference="caster_wheel">
     <mu1 value="1.0"/>
@@ -54,3 +63,21 @@
     <material>Gazebo/Black</material>
   </gazebo>
+  <gazebo reference="left_wall">
+    <material>Gazebo/Grey</material>
+    <mu1 value="1.0"/>
+    <mu2 value="1.0"/>
+    <kp  value="10000000.0"/>
+    <kd  value="100.0"/>
+    <maxVel>0.0</maxVel>
+    <minDepth>0.001</minDepth>
+  </gazebo>
+  <gazebo reference="right_wall">
+    <material>Gazebo/Grey</material>
+    <mu1 value="1.0"/>
+    <mu2 value="1.0"/>
+    <kp  value="10000000.0"/>
+    <kd  value="100.0"/>
+    <maxVel>0.0</maxVel>
+    <minDepth>0.001</minDepth>
+  </gazebo>
 </robot>

File: urdf/macros.xacro (robot description, xacro)
@@ -113,3 +113,29 @@
     </joint>
   </xacro:macro>
+  <xacro:macro name="guide_wall" params="side prefix">
+    <link name="${prefix}_wall">
+      <visual>
+        <geometry>
+          <box size="${wall_length} ${wall_thickness} ${wall_height}"/>
+        </geometry>
+        <material name="grey">
+          <color rgba="0.5 0.5 0.5 1"/>
+        </material>
+      </visual>
+      <collision>
+        <geometry>
+          <box size="${wall_length} ${wall_thickness} ${wall_height}"/>
+        </geometry>
+      </collision>
+      <inertial>
+        <mass value="0.3"/>
+        <inertia ixx="0.003" ixy="0" ixz="0" iyy="0.003" iyz="0" izz="0.003"/>
+      </inertial>
+   </link>
+   <joint name="${prefix}_wall_joint" type="fixed">
+      <parent link="base_link"/>
+      <child link="${prefix}_wall"/>
+      <origin xyz="${base_length/2 + wall_length/2} ${side * (base_width/2 + wall_thickness/2)} ${wall_height/2}" rpy="0 0 0"/>
+    </joint>
+  </xacro:macro>
 </robot>

File: urdf/properties.xacro (robot description, xacro)
@@ -10,3 +10,6 @@
   <xacro:property name="arm_length" value="0.1"/>
   <xacro:property name="arm_radius" value="0.015"/>
+  <xacro:property name="wall_length" value="0.3"/>
+  <xacro:property name="wall_thickness" value="0.01"/>
+  <xacro:property name="wall_height" value="0.16"/>
 </robot>

File: urdf/three_wheeled_robot.xacro (robot description, xacro)
@@ -33,5 +33,7 @@
   <xacro:wheel prefix="left" x="${-base_length/3}" y="1"/>
   <xacro:wheel prefix="right" x="${-base_length/3}" y="-1"/>
-  <xacro:arm prefix="left" side_mult="1"/>
-  <xacro:arm prefix="right" side_mult="-1"/>
+  <!-- <xacro:arm prefix="left" side_mult="1"/>
+  <xacro:arm prefix="right" side_mult="-1"/> -->
+  <xacro:guide_wall prefix="left" side="1"/>
+  <xacro:guide_wall prefix="right" side="-1"/>
 </robot>

Commit message: reduce inertia so that we dont send balls flying all over

File: urdf/gazebo.xacro (robot description, xacro)
@@ -17,8 +17,8 @@
       <publishOdomTF>true</publishOdomTF>
       <publishWheelJointState>true</publishWheelJointState>
-      <max_wheel_torque>20</max_wheel_torque>
-      <wheelAcceleration>1</wheelAcceleration>
-      <max_wheel_acceleration>1</max_wheel_acceleration>
-      <wheelTorque>20</wheelTorque>
+      <max_wheel_torque>10</max_wheel_torque>
+      <wheelAcceleration>0.5</wheelAcceleration>
+      <max_wheel_acceleration>0.5</max_wheel_acceleration>
+      <wheelTorque>10</wheelTorque>
       <updateRate>50</updateRate>
       <max_velocity>0.5</max_velocity>

File: urdf/macros.xacro (robot description, xacro)
@@ -130,5 +130,5 @@
       <inertial>
         <mass value="0.3"/>
-        <inertia ixx="0.003" ixy="0" ixz="0" iyy="0.003" iyz="0" izz="0.003"/>
+        <inertia ixx="0.001" ixy="0" ixz="0" iyy="0.001" iyz="0" izz="0.001"/>
       </inertial>
    </link>

File: urdf/three_wheeled_robot.xacro (robot description, xacro)
@@ -25,5 +25,5 @@
     </collision>
     <inertial>
-      <mass value="0.6"/>
+      <mass value="0.5"/>
       <inertia ixx="0.001" ixy="0" ixz="0" iyy="0.001" iyz="0" izz="0.001"/>
       <origin xyz="0 0 0" rpy="0 0 0"/>

Commit message: slam is done. works.

File: urdf/gazebo.xacro (robot description, xacro)
@@ -24,4 +24,30 @@
       <max_velocity>0.5</max_velocity>
     </plugin>
+  </gazebo>
+  <gazebo reference="laser_link">
+    <sensor type="ray" name="rplidar">
+      <pose>0 0 0 0 0 0</pose>
+      <visualize>true</visualize>
+      <update_rate>10</update_rate>
+      <ray>
+        <scan>
+          <horizontal>
+            <samples>360</samples>
+            <resolution>1</resolution>
+            <min_angle>-3.14159</min_angle>
+            <max_angle>3.14159</max_angle>
+          </horizontal>
+        </scan>
+        <range>
+          <min>0.1</min>
+          <max>6.0</max>
+          <resolution>0.01</resolution>
+        </range>
+      </ray>
+      <plugin name="gazebo_ros_rplidar_controller" filename="libgazebo_ros_laser.so">
+        <topicName>/scan</topicName>
+        <frameName>laser_link</frameName>
+      </plugin>
+    </sensor>
   </gazebo>
   <material name="orange">

File: urdf/properties.xacro (robot description, xacro)
@@ -13,3 +13,9 @@
   <xacro:property name="wall_thickness" value="0.01"/>
   <xacro:property name="wall_height" value="0.16"/>
+  <!-- LIDAR properties -->
+  <xacro:property name="lidar_cylinder_height" value="0.2"/>
+  <xacro:property name="lidar_radius" value="0.05"/>
+  <xacro:property name="lidar_height" value="0.05"/>
+  <xacro:property name="lidar_mount_x" value="0.0"/>
+  <xacro:property name="lidar_mount_y" value="0.0"/>
 </robot>

File: urdf/three_wheeled_robot.xacro (robot description, xacro)
@@ -8,4 +8,6 @@
   <!-- Include Gazebo configurations -->
   <xacro:include filename="$(find pde4430_coursework2)/urdf/gazebo.xacro" />
+  <!-- Include Lidar -->
+  <xacro:include filename="$(find pde4430_coursework2)/urdf/lidar.xacro" />
   <!-- Base Link -->
   <link name="base_link">
@@ -33,6 +35,4 @@
   <xacro:wheel prefix="left" x="${-base_length/3}" y="1"/>
   <xacro:wheel prefix="right" x="${-base_length/3}" y="-1"/>
-  <!-- <xacro:arm prefix="left" side_mult="1"/>
-  <xacro:arm prefix="right" side_mult="-1"/> -->
   <xacro:guide_wall prefix="left" side="1"/>
   <xacro:guide_wall prefix="right" side="-1"/>

File: urdf/twr.urdf (robot description, URDF)
Before this commit: robot three_wheeled_robot, 6 links, 5 joints
Links:
- added link laser_link, mass 0.1; collision cylinder length=0.05 radius=0.05; visual cylinder length=0.05 radius=0.05
- added link lidar_base_cylinder, mass 0.2; collision cylinder length=0.2 radius=0.02; visual cylinder length=0.2 radius=0.02
- link base_link: mass 0.6 -> 0.5; geometry collision box size=0.35 0.31 0.1; visual box size=0.35 0.31 0.05
Joints:
- added joint base_to_cylinder: type fixed, parent base_link, child lidar_base_cylinder, origin xyz=0 0 0.1 rpy=0 0 0
- added joint laser_joint: type fixed, parent lidar_base_cylinder, child laser_link, origin xyz=0.0 0.0 0.1 rpy=0 0 0
- joint left_wall_joint: origin xyz=0.32499999999999996 0.20500000000000002 0.08 rpy=0 0 0 -> xyz=0.32499999999999996 0.16 0.08 rpy=0 0 0
- joint left_wheel_joint: origin xyz=-0.11666666666666665 0.23500000000000001 0 rpy=1.5707963267948966 0 0 -> xyz=-0.11666666666666665 0.19 0 rpy=1.5707963267948966 0 0
- joint right_wall_joint: origin xyz=0.32499999999999996 -0.20500000000000002 0.08 rpy=0 0 0 -> xyz=0.32499999999999996 -0.16 0.08 rpy=0 0 0
- joint right_wheel_joint: origin xyz=-0.11666666666666665 -0.23500000000000001 0 rpy=1.5707963267948966 0 0 -> xyz=-0.11666666666666665 -0.19 0 rpy=1.5707963267948966 0 0
